File: power_section.kicad_sch (KiCad schematic)
At the start: 16 parts, among them J12 Conn_01x02_Pin, J13 Conn_01x05, J14 Conn_01x05, J15 Conn_01x05, J16 Conn_01x05, J17 Barrel_Jack, SW6 Slide Sw, U2 AMS1117-3.3, U3 MP1584 step down Module

Commit message: routing and gerber finished file
Parts:
- removed C11: 22uF, ~, symbol PCM_SparkFun-Capacitor:C_Polarized
- removed C9: 10uF, ~, symbol PCM_SparkFun-Capacitor:C_Polarized
- removed J13, J14, J15, J16: Conn_01x05, symbol Connector_Generic:Conn_01x05
- removed J17: Barrel_Jack, symbol Connector:Barrel_Jack
- added C1: 47uF/25V, Capacitor_THT:C_Radial_D5.0mm_H11.0mm_P2.00mm, symbol Device:C_Small_US
- added C2: 0.1 uF, Capacitor_THT:C_Disc_D5.0mm_W2.5mm_P2.50mm, symbol PCM_SparkFun-Capacitor:C
- added C3: 10uF, Capacitor_SMD:C_Elec_4x5.4, symbol Device:C_Small_US
- added C5: 22uF, Capacitor_SMD:C_Elec_5x5.4, symbol Device:C_Small_US
- added J1: Barrel_Jack, peripheral_lib:DCJack, symbol Connector:Barrel_Jack_MountingPin
- added J2: 5V_rail, Connector_PinHeader_2.54mm:PinHeader_2x05_P2.54mm_Vertical, symbol Connector_Generic:Conn_02x05_Counter_Clockwise
- added J3: 3.3V_rail, Connector_PinHeader_2.54mm:PinHeader_2x05_P2.54mm_Vertical, symbol Connector_Generic:Conn_02x05_Counter_Clockwise
- C4: renamed from C10; footprint PCM_SparkFun-Capacitor:C_0603_1608Metric -> Capacitor_THT:C_Disc_D5.0mm_W2.5mm_P2.50mm
- C6: renamed from C12; footprint PCM_SparkFun-Capacitor:C_0603_1608Metric -> Capacitor_THT:C_Disc_D5.0mm_W2.5mm_P2.50mm
- C7: renamed from C13; footprint PCM_SparkFun-Capacitor:C_0603_1608Metric -> Capacitor_SMD:C_1206_3216Metric_Pad1.33x1.80mm_HandSolder
- F1: footprint (none) -> Fuse:Fuse_Bourns_MF-RG400
- J6: renamed from J12; footprint (none) -> Connector_PinHeader_2.54mm:PinHeader_1x02_P2.54mm_Vertical
- JP1: renamed from JP2; footprint (none) -> Connector_PinHeader_2.54mm:PinHeader_1x03_P2.54mm_Vertical
- renumbered U3 to U1
Connections:
- net +3.3V: now also C5.1
- net +9V: now also J1.1
- net 5V: now also U1.3 (VCC-out), C3.1, J2.1 (Pin_1), J2.2 (Pin_2), J2.3 (Pin_3), J2.4 (Pin_4), J2.5 (Pin_5); no longer U1.4 (VCC-out)
- net GND: now also U1.1 (GND), U1.4 (GND), C1.2, C2.2, C3.2, C5.2, J1.2, J2.10 (Pin_10), J2.6 (Pin_6), J2.7 (Pin_7), J2.8 (Pin_8), J2.9 (Pin_9), J3.10 (Pin_10), J3.6 (Pin_6), J3.7 (Pin_7), J3.8 (Pin_8), J3.9 (Pin_9); no longer U1.2 (GND), U1.3 (GND)
- net at SW6.2 (B): now also J3.1 (Pin_1), J3.2 (Pin_2), J3.3 (Pin_3), J3.4 (Pin_4), J3.5 (Pin_5)
- net at F1.2: now also U1.2 (VCC-in), C1.1, C2.1; no longer U1.1 (VCC-in)
- no-connect marks 1 -> 2
Other:
- moved on the sheet: F1
